File: Hardware/ADCS/RWS.kicad_sch (KiCad schematic)
At the start: 0 parts

Commit message: ADCS PCB Schematic
Progress in Schematic
Added STM32 Project
Other:
- note added: "ADCS RWS"
- note added: "AMEYA MARAKARKANDY"
Changed lines of the file:
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@@
 	(generator_version "8.0")
 	(paper "A4")
+	(text "ADCS RWS"
+		(exclude_from_sim no)
+		(at 20.32 25.4 0)
+		(effects
+			(font
+				(size 5.08 5.08)
+				(thickness 0.508)
+				(bold yes)
+			)
+			(justify left bottom)
+		)
+	)
+	(text "AMEYA MARAKARKANDY"
+		(exclude_from_sim no)
+		(at 20.955 31.115 0)
+		(effects
+			(font
+				(size 2.54 2.54)
+				(bold yes)
+			)
+			(justify left bottom)
+		)
+	)
 )
