File: Hardware/ADCS/ADCS.kicad_pcb (KiCad board)
At the start: 2 copper layers, 92 x 92 mm, 41 parts, among them J1 Conn_02x26_Odd_Even, J2 Conn_02x26_Odd_Even, J3 USB_B_Micro, J4 Conn_01x04_Pin, SW1 SW_SPDT, U1 STM32L471VET6, U2 IIS2MDCTR, U3 BMI270, U4 AMS1117-3.3, U5 DRV8212P, U6 DRV8212P, U7 DRV8212P, Y1 32MHz

Commit message: ADCS PCB Schematic
Progress in Schematic
Added STM32 Project
Parts:
- added C17: 100nF, Capacitor_SMD:C_0603_1608Metric, F.Cu at (71.8, 97.8)
- added C18: 100nF, Capacitor_SMD:C_0603_1608Metric, F.Cu at (71.8, 100.3)
- added C19: 100nF, Capacitor_SMD:C_0603_1608Metric, F.Cu at (71.8, 102.9)
- added C20: 100nF, Capacitor_SMD:C_0603_1608Metric, F.Cu at (71.8, 105.4)
- added C21: 10uF, Capacitor_SMD:C_0603_1608Metric, F.Cu at (71.8, 107.9)
- added C22: 220nF, Capacitor_SMD:C_0603_1608Metric, F.Cu at (71.8, 110.4)
- added C23: 0.1uF, Capacitor_SMD:C_0603_1608Metric, F.Cu at (78.0, 51.0)
- added C24: 0.1uF, Capacitor_SMD:C_0603_1608Metric, F.Cu at (78.0, 53.6)
- added C25: 10uF, Capacitor_SMD:C_0603_1608Metric, F.Cu at (78.0, 56.1)
- added C26: 0.1uF, Capacitor_SMD:C_0603_1608Metric, F.Cu at (78.0, 58.6)
- added C27: 10uF, Capacitor_SMD:C_0603_1608Metric, F.Cu at (78.0, 61.1)
- added C28: 0.1uF, Capacitor_SMD:C_0603_1608Metric, F.Cu at (78.0, 63.6)
- added C29: 0.1uF, Capacitor_SMD:C_0603_1608Metric, F.Cu at (78.0, 66.1)
- added C30: 10uF, Capacitor_SMD:C_0603_1608Metric, F.Cu at (78.0, 68.6)
- added C31: 0.1uF, Capacitor_SMD:C_0603_1608Metric, F.Cu at (78.0, 71.1)
- added J5: Conn_01x04_Pin, Connector_PinHeader_2.54mm:PinHeader_1x04_P2.54mm_Horizontal, F.Cu at (84.4, 94.2)
- added Q1: PMOS, Package_TO_SOT_SMD:SOT-23-3, F.Cu at (84.9, 79.0)
- added Q2: PMOS, Package_TO_SOT_SMD:SOT-23-3, F.Cu at (84.9, 83.6)
- added R10: 0, Resistor_SMD:R_0603_1608Metric, F.Cu at (71.8, 92.9)
- added R4: 1k5, Resistor_SMD:R_0603_1608Metric, F.Cu at (71.8, 77.8)
- added R5: 1k5, Resistor_SMD:R_0603_1608Metric, F.Cu at (71.8, 80.3)
- added R6: 100k, Resistor_SMD:R_0603_1608Metric, F.Cu at (71.8, 82.8)
- added R7: 100, Resistor_SMD:R_0603_1608Metric, F.Cu at (71.8, 85.3)
- added R8: 100k, Resistor_SMD:R_0603_1608Metric, F.Cu at (71.8, 87.9)
- added R9: 100, Resistor_SMD:R_0603_1608Metric, F.Cu at (71.8, 90.4)
- added U10: TPS3824-33QDBVRQ1, TPS3824:tps3824, F.Cu at (102.0, 82.5)
- added U8: SN65HVD256D, SN65HVD:D8, F.Cu at (147.9, 66.0)
- added U9: SN65HVD256D, SN65HVD:D8, F.Cu at (155.6, 65.8)
- moved U7 119.6 mm to (82.2, 55.4)
- moved U6 119.4 mm to (82.2, 51.7)
- moved JP3 55.3 mm to (190.4, 69.4)
- moved JP2 55.3 mm to (185.8, 69.4)
- moved SW1 44.2 mm to (119.3, 70.3)
- moved J3 26.5 mm to (202.6, 76.6), turned to 90 degrees
- moved Y1 21.0 mm to (174.5, 123.6)
- moved 120R1 17.3 mm to (142.6, 115.3)
- moved C1 8.63 mm to (143.0, 99.4)
- moved D1 8.63 mm to (150.9, 94.8)
- moved R2 8.63 mm to (143.0, 106.9)
- moved C2 8.63 mm to (143.0, 101.9)
- moved D2 8.63 mm to (150.9, 97.8)
- moved R1 8.63 mm to (143.0, 104.4)
- moved J4 8.41 mm to (199.3, 60.1)
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Connections:
- U1 pad 70: unconnected-(U1-PA11-Pad70) -> /USB_D-
- U1 pad 71: unconnected-(U1-PA12-Pad71) -> /USB_D+
- U2 pad 1: unconnected-(U2-SCL/SPC-Pad1) -> /I2C_SCL
- U2 pad 10: unconnected-(U2-VDD_IO-Pad10) -> 3V3_ADCS
- U2 pad 3: unconnected-(U2-CS-Pad3) -> 3V3_ADCS
- U2 pad 4: unconnected-(U2-SDA/SDI/SDO-Pad4) -> /I2C_SDA
- U2 pad 5: unconnected-(U2-C1-Pad5) -> Net-(U2-C1)
- U2 pad 6: unconnected-(U2-GND-Pad6) -> GND
- U2 pad 7: unconnected-(U2-INT/DRDY-Pad7) -> /MAG_INT
- U2 pad 8: unconnected-(U2-GND-Pad8) -> GND
- U2 pad 9: unconnected-(U2-VDD-Pad9) -> 3V3_ADCS
- U3 pad 1: unconnected-(U3-SDO-Pad1) -> GND
- U3 pad 12: unconnected-(U3-CSB-Pad12) -> 3V3_ADCS
- U3 pad 13: unconnected-(U3-SCX-Pad13) -> /I2C_SCL
- U3 pad 14: unconnected-(U3-SDX-Pad14) -> /I2C_SDA
- U3 pad 4: unconnected-(U3-INT1-Pad4) -> /IMU_INT1
- U3 pad 5: unconnected-(U3-VDDIO-Pad5) -> 3V3_ADCS
- U3 pad 6: unconnected-(U3-GNDIO-Pad6) -> GND
- U3 pad 7: unconnected-(U3-GND-Pad7) -> GND
- U3 pad 8: unconnected-(U3-VDD-Pad8) -> 3V3_ADCS
- U3 pad 9: unconnected-(U3-INT2-Pad9) -> /IMU_INT2
- U5 pad 1: unconnected-(U5-VM-Pad1) -> 5V_ADCS
- U5 pad 2: unconnected-(U5-OUT1-Pad2) -> /MTQ/MTQX_1
- U5 pad 3: unconnected-(U5-OUT2-Pad3) -> /MTQ/MTQX_2
- U5 pad 4: Net-(U5-GND-Pad4) -> GND
- U5 pad 5: unconnected-(U5-IN2-Pad5) -> /IN2_MTQX
- U5 pad 6: unconnected-(U5-IN1-Pad6) -> /IN1_MTQX
- U5 pad 7: unconnected-(U5-~{SLEEP}-Pad7) -> /SLEEP_MTQX
- U5 pad 8: unconnected-(U5-VCC-Pad8) -> 3V3_ADCS
- U5 pad 9: Net-(U5-GND-Pad4) -> GND
- U6 pad 1: unconnected-(U6-VM-Pad1) -> 5V_ADCS
- U6 pad 2: unconnected-(U6-OUT1-Pad2) -> /MTQ/MTQY_1
- U6 pad 3: unconnected-(U6-OUT2-Pad3) -> /MTQ/MTQY_2
- U6 pad 4: Net-(U6-GND-Pad4) -> GND
- U6 pad 5: unconnected-(U6-IN2-Pad5) -> /IN2_MTQY
- U6 pad 6: unconnected-(U6-IN1-Pad6) -> /IN1_MTQY
- U6 pad 7: unconnected-(U6-~{SLEEP}-Pad7) -> /SLEEP_MTQY
- U6 pad 8: unconnected-(U6-VCC-Pad8) -> 3V3_ADCS
- U6 pad 9: Net-(U6-GND-Pad4) -> GND
- U7 pad 1: unconnected-(U7-VM-Pad1) -> 5V_ADCS
- U7 pad 2: unconnected-(U7-OUT1-Pad2) -> /MTQ/MTQZ_1
- U7 pad 3: unconnected-(U7-OUT2-Pad3) -> /MTQ/MTQZ_2
- U7 pad 4: Net-(U7-GND-Pad4) -> GND
- U7 pad 5: unconnected-(U7-IN2-Pad5) -> /IN2_MTQZ
- U7 pad 6: unconnected-(U7-IN1-Pad6) -> /IN1_MTQZ
- U7 pad 7: unconnected-(U7-~{SLEEP}-Pad7) -> /SLEEP_MTQZ
- U7 pad 8: unconnected-(U7-VCC-Pad8) -> 3V3_ADCS
- U7 pad 9: Net-(U7-GND-Pad4) -> GND
Other:
- copper layers 2 -> 4

Commit message: ADCS PCB Rough Layout
Parts:
- added U11: ~, MTQ:MTQ_ROD, F.Cu at (205.4, 127.8)
- added U12: ~, MTQ:MTQ_ROD, F.Cu at (113.3, 110.3)
- added U13: ~, MTQ:MTQ_AIRCORE, B.Cu at (159.3, 95.7)
- moved U5 141.7 mm to (39.0, 126.2)
- moved J3 86.3 mm to (116.3, 74.7), turned to -90 degrees
- moved U7 82.1 mm to (44.3, 128.2)
- moved U6 82.1 mm to (44.3, 124.5)
- moved D2 80.2 mm to (77.8, 130.7)
- moved D1 79.1 mm to (78.5, 126.7)
- moved J4 77.3 mm to (122.4, 67.4), turned to 180 degrees
- moved C1 75.7 mm to (68.6, 113.2)
- moved C2 75.7 mm to (68.6, 115.7)
- moved R1 75.7 mm to (68.6, 118.2)
- moved R2 75.7 mm to (68.6, 120.7)
- moved C8 74.8 mm to (216.5, 77.5)
- moved C10 69.8 mm to (225.8, 92.0)
- moved C3 69.8 mm to (221.7, 89.5)
- moved C9 69.8 mm to (225.8, 89.5)
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Routing:
- added copper zone on B.Cu, net GND
- added copper zone on F.Cu, net GND
