File: Hardware/ADCS/ADCS.kicad_sch (KiCad schematic)
At the start: 17 parts, among them J1 Conn_02x26_Odd_Even, J2 Conn_02x26_Odd_Even, J3 USB_B_Micro, J4 Conn_01x04_Pin, U4 AMS1117-3.3

Commit message: ADCS PCB Schematic
Progress in Schematic
Added STM32 Project
Other:
- sheet ControlUnit ports: added 3V3, CAN_A_H, CAN_A_L, CAN_B_H, CAN_B_L, GND, HEARTBEAT_ADCS, I2C_SCL, I2C_SDA, IMU_INT1, IMU_INT2, IN1_MTQX, IN1_MTQY, IN1_MTQZ, IN2_MTQX, IN2_MTQY, IN2_MTQZ, MAG_INT, SLEEP_MTQX, SLEEP_MTQY, SLEEP_MTQZ, SWCLK, SWDIO, UART_RX, UART_TX, USB_D+, USB_D-; removed none
- sheet MTQ ports: added 3V3, 5V, GND, IN1_MTQX, IN1_MTQY, IN1_MTQZ, IN2_MTQX, IN2_MTQY, IN2_MTQZ, SLEEP_MTQX, SLEEP_MTQY, SLEEP_MTQZ; removed none
- sheet Sensors ports: added 3V3, GND, I2C_SCL, I2C_SDA, IMU_INT1, IMU_INT2, MAG_INT, UART_RX, UART_TX; removed none
- moved on the sheet: J4, R2

Commit message: ADCS PCB Rough Layout
Other:
- note added: "M3"
- note removed: "M2"
Changed lines of the file:
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@@
 		)
 	)
-	(text "M2"
+	(text "M3"
 		(exclude_from_sim no)
 		(at 335.915 60.325 0)
