File: Hardware/ADCS/MTQ.kicad_sch (KiCad schematic)
At the start: 3 parts, among them U5 DRV8212P, U6 DRV8212P, U7 DRV8212P

Commit message: ADCS PCB Schematic
Progress in Schematic
Added STM32 Project
Parts:
- added C23, C24, C26, C28, C29, C31: 0.1uF, Capacitor_SMD:C_0603_1608Metric, symbol Device:C
- added C25, C27, C30: 10uF, Capacitor_SMD:C_0603_1608Metric, symbol Device:C
- added H10, H5, H6, H7, H8, H9: MountingHole_Pad, symbol Mechanical:MountingHole_Pad
- added L1, L2, L3: L, symbol Device:L
Connections:
- net +5V: now reaches U5.1 (VM)
- net +5V: now also U6.1 (VM), U7.1 (VM), C24.1, C25.1, C26.1, C27.1, C29.1, C30.1
- net MTQX_1: now reaches U5.2 (OUT1)
- net MTQX_1: now also L1.1
- net MTQX_2: now reaches U5.3 (OUT2)
- net MTQX_2: now also L1.2
- net GND: now reaches U5.4 (GND), U5.9 (GND)
- net GND: now also U6.4 (GND), U6.9 (GND), U7.4 (GND), U7.9 (GND), C23.2, C24.2, C25.2, C26.2, C27.2, C28.2, C29.2, C30.2, C31.2
- net IN2_MTQX: now reaches U5.5 (IN2)
- net IN1_MTQX: now reaches U5.6 (IN1)
- net SLEEP_MTQX: now reaches U5.7 (~{SLEEP})
- net +3.3V: now reaches U5.8 (VCC)
- net +3.3V: now also U6.8 (VCC), U7.8 (VCC), C23.1, C28.1, C31.1
- net MTQZ_1: now reaches U7.2 (OUT1)
- net MTQZ_1: now also L3.1
- net MTQZ_2: now reaches U7.3 (OUT2)
- net MTQZ_2: now also L3.2
- net IN2_MTQZ: now reaches U7.5 (IN2)
- net IN1_MTQZ: now reaches U7.6 (IN1)
- net SLEEP_MTQZ: now reaches U7.7 (~{SLEEP})
- net MTQY_1: now reaches U6.2 (OUT1)
- net MTQY_1: now also L2.1
- net MTQY_2: now reaches U6.3 (OUT2)
- net MTQY_2: now also L2.2
- net IN2_MTQY: now reaches U6.5 (IN2)
- net IN1_MTQY: now reaches U6.6 (IN1)
- net SLEEP_MTQY: now reaches U6.7 (~{SLEEP})
Other:
- note added: "ADCS MTQ"
- note added: "AMEYA MARAKARKANDY"
- note added: "MTQ_X"
- note added: "MTQ_Y"
- note added: "MTQ_Z"
- moved on the sheet: U5

Commit message: ADCS PCB Rough Layout
Parts:
- removed H10, H9: MountingHole_Pad, symbol Mechanical:MountingHole_Pad
- removed L1, L2, L3: L, symbol Device:L
- added U11, U12: ~, MTQ:MTQ_ROD, symbol MTQ:MTQ_ROD
- added U13: ~, MTQ:MTQ_AIRCORE, symbol MTQ:MTQ_AIRCORE
- H5, H6, H7, H8: footprint (none) -> MountingHole:MountingHole_2.2mm_M2_Pad
Connections:
- net GND: now also U11.3 (GND), U11.4 (GND), U12.3 (GND), U12.4 (GND), U13.3 (GND), U13.4 (GND), U13.5 (GND), U13.6 (GND)
- net MTQX_1: now also U13.1 (IN1)
- net MTQX_2: now also U13.2 (IN2)
- net MTQY_1: now also U12.1 (IN1)
- net MTQY_2: now also U12.2 (IN2)
- net MTQZ_1: now also U11.1 (IN1)
- net MTQZ_2: now also U11.2 (IN2)
Other:
- note removed: "MTQ_Y"
- moved on the sheet: H5, H6, H7, H8
