File: Hardware/ADCS/Sensors.kicad_sch (KiCad schematic)
At the start: 2 parts, among them U2 IIS2MDCTR, U3 BMI270

Commit message: ADCS PCB Schematic
Progress in Schematic
Added STM32 Project
Parts:
- added C17, C18, C19, C20: 100nF, Capacitor_SMD:C_0603_1608Metric, symbol Device:C
- added C21: 10uF, Capacitor_SMD:C_0603_1608Metric, symbol Device:C
- added C22: 220nF, Capacitor_SMD:C_0603_1608Metric, symbol Device:C
- added J5: Conn_01x04_Pin, Connector_PinHeader_2.54mm:PinHeader_1x04_P2.54mm_Horizontal, symbol Connector:Conn_01x04_Pin
Connections:
- net GND: now reaches U3.1 (SDO)
- net GND: now also U2.6 (GND), U2.8 (GND), U3.6 (GNDIO), U3.7 (GND), C17.2, C18.2, C19.2, C20.2, C21.2, C22.2, J5.4 (Pin_4)
- net +3.3V: now reaches U3.12 (CSB)
- net +3.3V: now also U2.10 (VDD_IO), U2.3 (CS), U2.9 (VDD), U3.5 (VDDIO), U3.8 (VDD), C17.1, C18.1, C19.1, C20.1, C21.1, J5.1 (Pin_1)
- net I2C_SCL: now reaches U3.13 (SCX)
- net I2C_SCL: now also U2.1 (SCL/SPC)
- net I2C_SDA: now reaches U3.14 (SDX)
- net I2C_SDA: now also U2.4 (SDA/SDI/SDO)
- net IMU_INT1: now reaches U3.4 (INT1)
- net IMU_INT2: now reaches U3.9 (INT2)
- net at U2.5 (C1): now also C22.1
- net MAG_INT: now reaches U2.7 (INT/DRDY)
- new net UART_RX: J5.3 (Pin_3)
- new net UART_TX: J5.2 (Pin_2)
- no-connect marks 0 -> 4
Other:
- note added: "ADCS SENSORS"
- note added: "AMEYA MARAKARKANDY"
- note added: "Default I2C Address (0x68) if SDO pin is pulled to GND"
- note added: "EXTERNAL CONNECTIONS"
- note added: "PULL UP RESISTORS ON I2C LINE ARE PROVIDED IN CONTROL UNIT"
- note added: "The following recommendations apply to capacitor C1:   It must be connected as close as possible to pins 5 and 6 since very high current pulses flow from C1 to pin 5 and 6. This avoids problems caused by inductive effects due to the length of the copper strips. It is highly recommended to use low ESR (max 200 mOhm)"
- moved on the sheet: U2, U3

Commit message: ADCS PCB Rough Layout
Other:
- note added: "MOLEX PICO LOCK"
Changed lines of the file:
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@@
+		)
+	)
+	(text "MOLEX PICO LOCK"
+		(exclude_from_sim no)
+		(at 198.12 154.432 0)
+		(effects
+			(font
+				(size 1.27 1.27)
+			)
 		)
 	)
